File: LightFusion.kicad_sch (KiCad schematic)
At the start: 54 parts, among them IC2 ADS1292IPBSR, U1 BMD-350-A-R, U4 DRV8837DSGR

Commit message: refined electrodes symb
Parts:
- E_EEG1, E_EEG2, E_EEG3, STIM_E_N1, STIM_E_P1: symbol Electrode_MillMax_0906:Electrode_MillMax_0906 -> Electrode:Electrode_MillMax_0906
Changed lines of the file:
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@@
 	)
 	(symbol
-		(lib_id "Electrode_MillMax_0906:Electrode_MillMax_0906")
+		(lib_name "Electrode_MillMax_0906_4")
+		(lib_id "Electrode:Electrode_MillMax_0906")
 		(at 166.37 82.55 0)
 		(unit 1)
@@
 	)
 	(symbol
-		(lib_id "Electrode_MillMax_0906:Electrode_MillMax_0906")
+		(lib_name "Electrode_MillMax_0906_2")
+		(lib_id "Electrode:Electrode_MillMax_0906")
 		(at 147.32 160.02 0)
 		(unit 1)
@@
 	)
 	(symbol
-		(lib_id "Electrode_MillMax_0906:Electrode_MillMax_0906")
+		(lib_name "Electrode_MillMax_0906_3")
+		(lib_id "Electrode:Electrode_MillMax_0906")
 		(at 167.64 114.3 0)
 		(unit 1)
@@
 	)
 	(symbol
-		(lib_id "Electrode_MillMax_0906:Electrode_MillMax_0906")
+		(lib_name "Electrode_MillMax_0906_1")
+		(lib_id "Electrode:Electrode_MillMax_0906")
 		(at 142.24 153.67 0)
 		(unit 1)
@@
 	)
 	(symbol
-		(lib_id "Electrode_MillMax_0906:Electrode_MillMax_0906")
+		(lib_id "Electrode:Electrode_MillMax_0906")
 		(at 177.8 72.39 0)
 		(unit 1)

Commit message: another electrode symb adjustment
Parts:
- E_EEG1, E_EEG2, E_EEG3, STIM_E_N1, STIM_E_P1: symbol Electrode:Electrode_MillMax_0906 -> Electrode_MillMax_0906:Electrode_MillMax_0906
Changed lines of the file:
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@@
 	)
 	(symbol
-		(lib_name "Electrode_MillMax_0906_4")
-		(lib_id "Electrode:Electrode_MillMax_0906")
+		(lib_id "Electrode_MillMax_0906:Electrode_MillMax_0906")
 		(at 166.37 82.55 0)
 		(unit 1)
@@
 	)
 	(symbol
-		(lib_name "Electrode_MillMax_0906_2")
-		(lib_id "Electrode:Electrode_MillMax_0906")
+		(lib_id "Electrode_MillMax_0906:Electrode_MillMax_0906")
 		(at 147.32 160.02 0)
 		(unit 1)
@@
 	)
 	(symbol
-		(lib_name "Electrode_MillMax_0906_3")
-		(lib_id "Electrode:Electrode_MillMax_0906")
+		(lib_id "Electrode_MillMax_0906:Electrode_MillMax_0906")
 		(at 167.64 114.3 0)
 		(unit 1)
@@
 	)
 	(symbol
-		(lib_name "Electrode_MillMax_0906_1")
-		(lib_id "Electrode:Electrode_MillMax_0906")
+		(lib_id "Electrode_MillMax_0906:Electrode_MillMax_0906")
 		(at 142.24 153.67 0)
 		(unit 1)
@@
 	)
 	(symbol
-		(lib_id "Electrode:Electrode_MillMax_0906")
+		(lib_id "Electrode_MillMax_0906:Electrode_MillMax_0906")
 		(at 177.8 72.39 0)
 		(unit 1)
