File: PD_ADC.kicad_sch (KiCad schematic)
At the start: 22 parts

Commit message: placement finished on PCB
Parts:
- removed U_ADC1: MCP3564R-E_ST, LightFusion:MCP3561T-E_NC, symbol MCP3561T-E_NC:MCP3561T-E_NC
- added IC1: MCP3561T-E_ST, LightFusion:MCP3561T-E_ST, symbol MCP3561T-E_ST:MCP3561T-E_ST
- C_ADC_AVDD_BULK1, C_ADC_AVDD_BYP1, C_ADC_DVDD_BULK1, C_ADC_DVDD_BYP1, C_ADC_PHOTO_N1, C_ADC_PHOTO_P1, C_ADC_REF_BULK1, C_ADC_REF_BYP1, C_PD_BIAS1, C_PD_FB1, C_PD_TIA_SUPPLY1: footprint (none) -> LightFusion:C_0603_1608Metric
- R_ADC_CS_PU1, R_ADC_IRQ_PU1, R_ADC_PHOTO_N1, R_ADC_PHOTO_P1, R_PD_BIAS_BOT1, R_PD_BIAS_TOP1, R_PD_FB1, R_PD_SUPPLY1: footprint (none) -> LightFusion:R_0603_1608Metric
Connections:
- net 3V3_A: now also IC1.1 (AVDD)
- net 3V3_DIG: now also IC1.20 (DVDD)
- net ADC_CS_N: now also IC1.13 (~{CS})
- net ADC_DRDY_N: now also IC1.17 (~{IRQ}/MDAT)
- net ADC_MISO: now also IC1.16 (SDO)
- net ADC_MOSI: now also IC1.15 (SDI)
- net ADC_PHOTO_N: now also IC1.6 (CH1)
- net ADC_PHOTO_P: now also IC1.5 (CH0)
- net ADC_SCK: now also IC1.14 (SCK)
- net ADC_VREF: now also IC1.4 (REFIN+)
- net GND: now also IC1.10 (NC_4), IC1.11 (NC_5), IC1.12 (NC_6), IC1.19 (DGND), IC1.2 (AGND), IC1.3 (REFIN-), IC1.7 (NC_1), IC1.8 (NC_2), IC1.9 (NC_3)

Commit message: final verifications
Changed lines of the file:
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@@
 		(fields_autoplaced yes)
 		(property "Reference" "C_ADC_PHOTO_P1"
-			(at 143.51 90.2969 0)
+			(at 143.51 91.5669 0)
 			(show_name no)
 			(do_not_autoplace no)
@@
 		(fields_autoplaced yes)
 		(property "Reference" "C_ADC_DVDD_BYP1"
-			(at 199.39 38.2269 0)
+			(at 199.39 39.4969 0)
 			(show_name no)
 			(do_not_autoplace no)
@@
 		(fields_autoplaced yes)
 		(property "Reference" "C_ADC_PHOTO_N1"
-			(at 134.62 86.4869 0)
+			(at 134.62 87.7569 0)
 			(show_name no)
 			(do_not_autoplace no)
@@
 		(fields_autoplaced yes)
 		(property "Reference" "C_ADC_DVDD_BULK1"
-			(at 205.74 45.8469 0)
+			(at 205.74 47.1169 0)
 			(show_name no)
 			(do_not_autoplace no)
@@
 		(fields_autoplaced yes)
 		(property "Reference" "C_PD_BIAS1"
-			(at 50.8 71.2469 0)
+			(at 50.8 72.5169 0)
 			(show_name no)
 			(do_not_autoplace no)
@@
 		(fields_autoplaced yes)
 		(property "Reference" "C_ADC_AVDD_BULK1"
-			(at 146.05 38.2269 0)
+			(at 146.05 39.4969 0)
 			(show_name no)
 			(do_not_autoplace no)
@@
 		(fields_autoplaced yes)
 		(property "Reference" "C_ADC_AVDD_BYP1"
-			(at 151.13 45.8469 0)
+			(at 151.13 47.1169 0)
 			(show_name no)
 			(do_not_autoplace no)
@@
 		(fields_autoplaced yes)
 		(property "Reference" "C_PD_FB1"
-			(at 111.76 67.4369 0)
+			(at 111.76 68.7069 0)
 			(show_name no)
 			(do_not_autoplace no)
@@
 		(fields_autoplaced yes)
 		(property "Reference" "C_PD_TIA_SUPPLY1"
-			(at 97.79 34.4169 0)
-			(show_name no)
-			(do_not_autoplace no)
+			(at 97.79 35.6869 0)
+			(show_name no)
+			(do_not_autoplace no)

Commit message: sync with available parts on JLC
Parts:
- C_ADC_PHOTO_N1, C_ADC_PHOTO_P1: footprint LightFusion:C_0603_1608Metric -> LightFusion:C_1206_3216Metric
Changed lines of the file:
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@@
 			)
 		)
-		(property "Footprint" "LightFusion:C_0603_1608Metric"
+		(property "Footprint" "LightFusion:C_1206_3216Metric"
 			(at 140.97 91.44 0)
 			(hide yes)
@@
 			)
 		)
-		(property "Footprint" "LightFusion:C_0603_1608Metric"
+		(property "Footprint" "LightFusion:C_1206_3216Metric"
 			(at 132.08 87.63 0)
 			(hide yes)
@@
 			)
 		)
-		(property "Description" "capacitor, small US symbol"
+		(property "Description" ""
 			(at 132.08 87.63 0)
 			(hide yes)

Commit message: final version with bom and placement
Parts:
- renumbered C_ADC_AVDD_BULK1 to C33, C_ADC_AVDD_BYP1 to C34, C_ADC_DVDD_BULK1 to C35, C_ADC_DVDD_BYP1 to C36, C_ADC_PHOTO_N1 to C37, C_ADC_PHOTO_P1 to C38, C_ADC_REF_BULK1 to C39, C_ADC_REF_BYP1 to C40, C_PD_BIAS1 to C41, C_PD_FB1 to C42, C_PD_TIA_SUPPLY1 to C43, D_PD1 to D3, R_ADC_CS_PU1 to R28, R_ADC_IRQ_PU1 to R29, R_ADC_PHOTO_N1 to R30, R_ADC_PHOTO_P1 to R31, R_PD_BIAS_BOT1 to R32, R_PD_BIAS_TOP1 to R33, R_PD_FB1 to R34, R_PD_SUPPLY1 to R35, U_PD_TIA1 to U10, IC1 to U9
Changed lines of the file:
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@@
 		(dnp no)
 		(fields_autoplaced yes)
-		(property "Reference" "C_ADC_PHOTO_P1"
+		(property "Reference" "C38"
 			(at 143.51 91.5669 0)
 			(show_name no)
@@
 			(project "LightFusion"
 				(path "/1aacc45f-6fcc-4559-bec0-55c6f50555c1/4857c65e-20bc-4a2b-a736-d87169b52ac1"
-					(reference "C_ADC_PHOTO_P1")
+					(reference "C38")
 					(unit 1)
 				)
@@
 		(dnp no)
 		(fields_autoplaced yes)
-		(property "Reference" "R_PD_BIAS_TOP1"
+		(property "Reference" "R33"
 			(at 67.31 43.1799 0)
 			(show_name no)
@@
 			(project "LightFusion"
 				(path "/1aacc45f-6fcc-4559-bec0-55c6f50555c1/4857c65e-20bc-4a2b-a736-d87169b52ac1"
-					(reference "R_PD_BIAS_TOP1")
+					(reference "R33")
 					(unit 1)
 				)
@@
 		(dnp no)
 		(fields_autoplaced yes)
-		(property "Reference" "C_ADC_DVDD_BYP1"
+		(property "Reference" "C36"
 			(at 199.39 39.4969 0)
 			(show_name no)
@@
 			(project "LightFusion"
 				(path "/1aacc45f-6fcc-4559-bec0-55c6f50555c1/4857c65e-20bc-4a2b-a736-d87169b52ac1"
-					(reference "C_ADC_DVDD_BYP1")
+					(reference "C36")
 					(unit 1)
 				)
@@
 		(in_pos_files yes)
 		(dnp no)
-		(fields_autoplaced yes)
-		(property "Reference" "R_ADC_PHOTO_P1"
-			(at 125.73 53.34 90)
+		(property "Reference" "R31"
+			(at 124.46 57.15 90)
 			(show_name no)
 			(do_not_autoplace no)
@@
 			(project "LightFusion"
 				(path "/1aacc45f-6fcc-4559-bec0-55c6f50555c1/4857c65e-20bc-4a2b-a736-d87169b52ac1"
-					(reference "R_ADC_PHOTO_P1")
+					(reference "R31")
 					(unit 1)
 				)
@@
 		(dnp no)
 		(fields_autoplaced yes)
-		(property "Reference" "C_ADC_PHOTO_N1"
+		(property "Reference" "C37"
 			(at 134.62 87.7569 0)
 			(show_name no)
@@
 			(project "LightFusion"
 				(path "/1aacc45f-6fcc-4559-bec0-55c6f50555c1/4857c65e-20bc-4a2b-a736-d87169b52ac1"
-					(reference "C_ADC_PHOTO_N1")
+					(reference "C37")
 					(unit 1)
 				)
@@
 		(in_pos_files yes)
 		(dnp no)
-		(property "Reference" "C_ADC_REF_BULK1"
-			(at 143.51 58.42 0)
+		(property "Reference" "C39"
+			(at 146.05 55.88 0)
 			(show_name no)
 			(do_not_autoplace no)
@@
 			(project "LightFusion"
 				(path "/1aacc45f-6fcc-4559-bec0-55c6f50555c1/4857c65e-20bc-4a2b-a736-d87169b52ac1"
-					(reference "C_ADC_REF_BULK1")
+					(reference "C39")
 					(unit 1)
 				)
@@
 		(dnp no)
 		(fields_autoplaced yes)
-		(property "Reference" "D_PD1"
+		(property "Reference" "D3"
 			(at 113.03 95.25 0)
 			(show_name no)
@@
 			(project "LightFusion"
 				(path "/1aacc45f-6fcc-4559-bec0-55c6f50555c1/4857c65e-20bc-4a2b-a736-d87169b52ac1"
-					(reference "D_PD1")
+					(reference "D3")
 					(unit 1)
 				)
@@
 		(dnp no)
 		(fields_autoplaced yes)
-		(property "Reference" "C_ADC_DVDD_BULK1"
+		(property "Reference" "C35"
 			(at 205.74 47.1169 0)
 			(show_name no)
@@
 			(project "LightFusion"
 				(path "/1aacc45f-6fcc-4559-bec0-55c6f50555c1/4857c65e-20bc-4a2b-a736-d87169b52ac1"
-					(reference "C_ADC_DVDD_BULK1")
+					(reference "C35")
 					(unit 1)
 				)
@@
 		(dnp no)
 		(fields_autoplaced yes)
-		(property "Reference" "C_PD_BIAS1"
+		(property "Reference" "C41"
 			(at 50.8 72.5169 0)
 			(show_name no)
@@
 			(project "LightFusion"
 				(path "/1aacc45f-6fcc-4559-bec0-55c6f50555c1/4857c65e-20bc-4a2b-a736-d87169b52ac1"
-					(reference "C_PD_BIAS1")
+					(reference "C41")
 					(unit 1)
 				)
@@
 		(dnp no)
 		(fields_autoplaced yes)
-		(property "Reference" "R_PD_FB1"
+		(property "Reference" "R34"
 			(at 125.73 67.3099 0)
 			(show_name no)
@@
 			(project "LightFusion"
 				(path "/1aacc45f-6fcc-4559-bec0-55c6f50555c1/4857c65e-20bc-4a2b-a736-d87169b52ac1"
-					(reference "R_PD_FB1")
+					(reference "R34")
 					(unit 1)
 				)
@@
 		(dnp no)
 		(fields_autoplaced yes)
-		(property "Reference" "C_ADC_AVDD_BULK1"
+		(property "Reference" "C33"
 			(at 146.05 39.4969 0)
 			(show_name no)
@@
 			(project "LightFusion"
 				(path "/1aacc45f-6fcc-4559-bec0-55c6f50555c1/4857c65e-20bc-4a2b-a736-d87169b52ac1"
-					(reference "C_ADC_AVDD_BULK1")
+					(reference "C33")
 					(unit 1)
 				)
@@
 		(in_pos_files yes)
 		(dnp no)
-		(fields_autoplaced yes)
-		(property "Reference" "R_PD_BIAS_BOT1"
-			(at 67.31 72.3899 0)
+		(property "Reference" "R32"
+			(at 60.96 71.12 0)
 			(show_name no)
 			(do_not_autoplace no)
@@
 			(project "LightFusion"
 				(path "/1aacc45f-6fcc-4559-bec0-55c6f50555c1/4857c65e-20bc-4a2b-a736-d87169b52ac1"
-					(reference "R_PD_BIAS_BOT1")
+					(reference "R32")
 					(unit 1)
 				)
@@
 		(dnp no)
 		(fields_autoplaced yes)
-		(property "Reference" "R_ADC_IRQ_PU1"
+		(property "Reference" "R29"
 			(at 224.79 74.9299 0)
 			(show_name no)
@@
 			(project "LightFusion"
 				(path "/1aacc45f-6fcc-4559-bec0-55c6f50555c1/4857c65e-20bc-4a2b-a736-d87169b52ac1"
-					(reference "R_ADC_IRQ_PU1")
+					(reference "R29")
 					(unit 1)
 				)
@@
 		(dnp no)
 		(fields_autoplaced yes)
-		(property "Reference" "C_ADC_AVDD_BYP1"
+		(property "Reference" "C34"
 			(at 151.13 47.1169 0)
 			(show_name no)
@@
 			(project "LightFusion"
 				(path "/1aacc45f-6fcc-4559-bec0-55c6f50555c1/4857c65e-20bc-4a2b-a736-d87169b52ac1"
-					(reference "C_ADC_AVDD_BYP1")
+					(reference "C34")
 					(unit 1)
 				)
@@
 		(dnp no)
 		(fields_autoplaced yes)
-		(property "Reference" "C_PD_FB1"
+		(property "Reference" "C42"
 			(at 111.76 68.7069 0)
 			(show_name no)
@@
 			(project "LightFusion"
 				(path "/1aacc45f-6fcc-4559-bec0-55c6f50555c1/4857c65e-20bc-4a2b-a736-d87169b52ac1"
-					(reference "C_PD_FB1")
+					(reference "C42")
 					(unit 1)
 				)
@@
 		(in_pos_files yes)
 		(dnp no)
-		(property "Reference" "C_ADC_REF_BYP1"
+		(property "Reference" "C40"
 			(at 158.75 55.88 0)
 			(show_name no)
@@
 			(project "LightFusion"
 				(path "/1aacc45f-6fcc-4559-bec0-55c6f50555c1/4857c65e-20bc-4a2b-a736-d87169b52ac1"
-					(reference "C_ADC_REF_BYP1")
+					(reference "C40")
 					(unit 1)
 				)
@@
 		(dnp no)
 		(fields_autoplaced yes)
-		(property "Reference" "C_PD_TIA_SUPPLY1"
+		(property "Reference" "C43"
 			(at 97.79 35.6869 0)
 			(show_name no)
@@
 			(project "LightFusion"
 				(path "/1aacc45f-6fcc-4559-bec0-55c6f50555c1/4857c65e-20bc-4a2b-a736-d87169b52ac1"
-					(reference "C_PD_TIA_SUPPLY1")
+					(reference "C43")
 					(unit 1)
 				)
@@
 		(in_pos_files yes)
 		(dnp no)
-		(property "Reference" "R_ADC_PHOTO_N1"
+		(property "Reference" "R30"
 			(at 82.55 81.28 90)
 			(show_name no)
@@
 			(project "LightFusion"
 				(path "/1aacc45f-6fcc-4559-bec0-55c6f50555c1/4857c65e-20bc-4a2b-a736-d87169b52ac1"
-					(reference "R_ADC_PHOTO_N1")
+					(reference "R30")
 					(unit 1)
 				)
@@
 		(dnp no)
 		(fields_autoplaced yes)
-		(property "Reference" "U_PD_TIA1"
+		(property "Reference" "U10"
 			(at 87.63 54.61 0)
 			(show_name no)
@@
 			(project "LightFusion"
 				(path "/1aacc45f-6fcc-4559-bec0-55c6f50555c1/4857c65e-20bc-4a2b-a736-d87169b52ac1"
-					(reference "U_PD_TIA1")
+					(reference "U10")
 					(unit 1)
 				)
@@
 		(dnp no)
 		(fields_autoplaced yes)
-		(property "Reference" "IC1"
+		(property "Reference" "U9"
 			(at 196.85 80.01 0)
 			(show_name no)
@@
 			(project "LightFusion"
 				(path "/1aacc45f-6fcc-4559-bec0-55c6f50555c1/4857c65e-20bc-4a2b-a736-d87169b52ac1"
-					(reference "IC1")
+					(reference "U9")
 					(unit 1)
 				)
@@
 		(dnp no)
 		(fields_autoplaced yes)
-		(property "Reference" "R_ADC_CS_PU1"
+		(property "Reference" "R28"
 			(at 224.79 64.7699 0)
 			(show_name no)
@@
 			(project "LightFusion"
 				(path "/1aacc45f-6fcc-4559-bec0-55c6f50555c1/4857c65e-20bc-4a2b-a736-d87169b52ac1"
-					(reference "R_ADC_CS_PU1")
+					(reference "R28")
 					(unit 1)
 				)
@@
 		(dnp no)
 		(fields_autoplaced yes)
-		(property "Reference" "R_PD_SUPPLY1"
+		(property "Reference" "R35"
 			(at 218.44 27.9399 0)
 			(show_name no)
@@
 			(project "LightFusion"
 				(path "/1aacc45f-6fcc-4559-bec0-55c6f50555c1/4857c65e-20bc-4a2b-a736-d87169b52ac1"
-					(reference "R_PD_SUPPLY1")
-					(unit 1)
-				)
+					(reference "R35")
+					(unit 1)
+				)
