File: PD_ADC.kicad_sch (KiCad schematic)
At the start: 22 parts, among them U10 OPA381AIDGKR, U9 MCP3561T-E_ST

Commit message: routing ready DRC passed
Parts:
- D3: footprint LightFusion:VEMD8082 -> LightFusion:VEMD8082_New; symbol VEMD8082:VEMD8082 -> VEMD8082_New:VEMD8082
Changed lines of the file:
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@@
 	)
 	(symbol
-		(lib_id "VEMD8082:VEMD8082")
+		(lib_id "VEMD8082_New:VEMD8082")
 		(at 92.71 102.87 0)
 		(unit 1)
@@
 		(fields_autoplaced yes)
 		(property "Reference" "D3"
-			(at 113.03 95.25 0)
+			(at 113.03 97.79 0)
 			(show_name no)
 			(do_not_autoplace no)
@@
 			)
 		)
-		(property "Footprint" "LightFusion:VEMD8082"
+		(property "Footprint" "LightFusion:VEMD8082_New"
 			(at 129.54 197.79 0)
 			(hide yes)

Commit message: 3d model ready
Parts:
- added J3, J4, J5, J6: Conn_01x01_Pin, LightFusion:TestPoint_THTPad_1.5x1.5mm_Drill0.7mm, symbol Conn_01x01_Pin:Conn_01x01_Pin
- D3: footprint LightFusion:VEMD8082_New -> LightFusion:VEMD8082C
Connections:
- net GND: now also J6.1 (Pin_1)
- net PHOTO_TIA_IN: now also J3.1 (Pin_1), J4.1 (Pin_1), J5.1 (Pin_1)

Commit message: daughter tmp board
Changed lines of the file:
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@@
 	)
 	(symbol
+		(lib_name "Conn_01x01_Pin_1")
 		(lib_id "Conn_01x01_Pin:Conn_01x01_Pin")
 		(at 87.63 110.49 0)
@@
 	)
 	(symbol
+		(lib_name "Conn_01x01_Pin_3")
 		(lib_id "Conn_01x01_Pin:Conn_01x01_Pin")
 		(at 138.43 102.87 180)
@@
 		(property "Reference" "J5"
 			(at 137.795 100.33 0)
+			(hide yes)
 			(show_name no)
 			(do_not_autoplace no)
@@
 	)
 	(symbol
+		(lib_name "Conn_01x01_Pin_2")
 		(lib_id "Conn_01x01_Pin:Conn_01x01_Pin")
 		(at 146.05 110.49 180)
