File: Power.kicad_sch (KiCad schematic)
At the start: 10 parts, among them J1 303C-C4115-30-04, P1 PHR-2, U2 TPS7A2033PDBVR, U3 TPS22918DBVR

Commit message: final version with bom and placement
Parts:
- renumbered C_PWR3 to C23, C_PWR4 to C24, C_PWR_SW_CT1 to C25, R_ON_PD1 to R24
Changed lines of the file:
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@@
 		(in_pos_files yes)
 		(dnp no)
-		(fields_autoplaced yes)
-		(property "Reference" "C_PWR4"
-			(at 173.99 73.7869 0)
+		(property "Reference" "C24"
+			(at 172.72 73.66 0)
 			(show_name no)
 			(do_not_autoplace no)
@@
 		(property "Value" "1 uF"
 			(at 173.99 76.3269 0)
+			(hide yes)
 			(show_name no)
 			(do_not_autoplace no)
@@
 			(project "LightFusion"
 				(path "/1aacc45f-6fcc-4559-bec0-55c6f50555c1/5e0cd53b-8700-46c2-b7ce-d555894c5a40"
-					(reference "C_PWR4")
+					(reference "C24")
 					(unit 1)
 				)
@@
 		(dnp no)
 		(fields_autoplaced yes)
-		(property "Reference" "C_PWR3"
+		(property "Reference" "C23"
 			(at 129.54 72.5169 0)
 			(show_name no)
@@
 			(project "LightFusion"
 				(path "/1aacc45f-6fcc-4559-bec0-55c6f50555c1/5e0cd53b-8700-46c2-b7ce-d555894c5a40"
-					(reference "C_PWR3")
+					(reference "C23")
 					(unit 1)
 				)
@@
 		(in_pos_files yes)
 		(dnp no)
-		(fields_autoplaced yes)
-		(property "Reference" "R_ON_PD1"
-			(at 110.49 110.4899 0)
+		(property "Reference" "R24"
+			(at 109.22 110.49 0)
 			(show_name no)
 			(do_not_autoplace no)
@@
 			(project "LightFusion"
 				(path "/1aacc45f-6fcc-4559-bec0-55c6f50555c1/5e0cd53b-8700-46c2-b7ce-d555894c5a40"
-					(reference "R_ON_PD1")
+					(reference "R24")
 					(unit 1)
 				)
@@
 		(dnp no)
 		(fields_autoplaced yes)
-		(property "Reference" "C_PWR_SW_CT1"
+		(property "Reference" "C25"
 			(at 152.4 114.4269 0)
 			(show_name no)
@@
 			(project "LightFusion"
 				(path "/1aacc45f-6fcc-4559-bec0-55c6f50555c1/5e0cd53b-8700-46c2-b7ce-d555894c5a40"
-					(reference "C_PWR_SW_CT1")
-					(unit 1)
-				)
+					(reference "C25")
+					(unit 1)
+				)
