File: LED.kicad_sch (KiCad schematic)
At the start: 15 parts, among them U6 STCS1APHR_FIXED, U7 STCS1APHR_FIXED, U8 TMP1075NDRLR

Commit message: new rect version
Parts:
- removed C30, C31: 10 nF, LightFusion:C_0603_1608Metric, symbol C_Small_US:C_Small_US
- added OPT1, OPT2: FP11055_LISA2-RS-PIN, LightFusion:LEDIL_FP11055_LISA2_RS_PIN, symbol LEDIL_FP11055_LISA2_RS_PIN:FP11055_LISA2_RS_PIN
- added R36: 100k, LightFusion:R_0603_1608Metric, symbol R_Small_US:R_Small_US
- added R37: 100k, LightFusion:R_1206_3216Metric, symbol R_Small_US:R_Small_US
- C26, C28: value 4.7 uF -> 10 uF
- U6, U7: value STCS1APHR_FIXED -> (none); footprint LightFusion:STCS1APHR-8_STM -> LightFusion:PAM2808BLBR; symbol STCS1APHR:STCS1APHR_FIXED -> PAM2808BLBR:PAM2808BLBR
Connections:
- net 3V3_DIG: no longer U6.3 (EN), U7.3 (EN)
- net GND: now also U6.4 (GND), U6.9 (GND), U7.4 (GND), U7.9 (GND), R36.2, R37.2; no longer U6.6 (GND), U6.EPAD, U7.6 (GND), U7.EPAD
- net PWM_730: now also U6.3 (EN), R37.1; no longer U6.2 (PWM)
- net PWM_850: now also U7.3 (EN), R36.1; no longer U7.2 (PWM)
- net VBAT_SYSTEM: now also U6.2 (VIN), U7.2 (VIN); no longer D1.2 (A), D2.2 (A), U6.1 (VCC), U7.1 (VCC)
- net at U7.7 (VOUT): now also D2.2 (A)
- net at U6.7 (VOUT): now also D1.2 (A)
- net at R25.1: now also D1.1 (K), U6.6 (FB); no longer U6.5 (FB)
- net at R26.1: now also D2.1 (K), U7.6 (FB); no longer U7.5 (FB)
- removed net LED730_K: D1.1 (K), U6.4 (DRAIN)
- removed net LED850_K: D2.1 (K), U7.4 (DRAIN)
- no-connect marks 2 -> 0
Other:
- moved on the sheet: D1, R25, R26

Commit message: rectangle placement
Parts:
- R37: footprint LightFusion:R_1206_3216Metric -> LightFusion:R_0603_1608Metric
Changed lines of the file:
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@@
 			)
 		)
-		(property "Footprint" "LightFusion:R_1206_3216Metric"
+		(property "Footprint" "LightFusion:R_0603_1608Metric"
 			(at 86.36 96.52 0)
 			(hide yes)
