File: TMP_Daughterboard/TMP_Daughterboard.kicad_sch (KiCad schematic)
At the start: 1 part, among them U1 TMP1075NDRLR

Commit message: daughter tmp board
Parts:
- U1: footprint TMP_Daughterboard:TMP1075-MOD-A -> TMP_Daughterboard:TMP1075-MOD-B
Connections:
- net at U1.2 (GND): now also U1.4 (A0)
Changed lines of the file:
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@@
 	(generator_version "10.0")
 	(paper "A4")
+	(wire
+		(pts
+			(xy 167.64 96.52) (xy 158.75 96.52)
+		)
+		(stroke
+			(width 0)
+			(type default)
+		)
+	)
+	(wire
+		(pts
+			(xy 124.46 80.01) (xy 124.46 64.77)
+		)
+		(stroke
+			(width 0)
+			(type default)
+		)
+	)
+	(wire
+		(pts
+			(xy 124.46 64.77) (xy 167.64 64.77)
+		)
+		(stroke
+			(width 0)
+			(type default)
+		)
+	)
+	(wire
+		(pts
+			(xy 167.64 64.77) (xy 167.64 96.52)
+		)
+		(stroke
+			(width 0)
+			(type default)
+		)
+	)
+	(wire
+		(pts
+			(xy 158.75 90.17) (xy 160.02 90.17)
+		)
+		(stroke
+			(width 0)
+			(type default)
+		)
+	)
+	(wire
+		(pts
+			(xy 158.75 96.52) (xy 158.75 90.17)
+		)
+		(stroke
+			(width 0)
+			(type default)
+		)
+	)
 	(symbol
 		(lib_id "TMP1075NDRLR:TMP1075NDRLR")
@@
 			)
 		)
-		(property "Footprint" "TMP_Daughterboard:TMP1075-MOD-A"
+		(property "Footprint" "TMP_Daughterboard:TMP1075-MOD-B"
 			(at 142.24 82.55 0)
 			(hide yes)
